Commit message: Add compatibility to ROS indigo

File: labrob_description/urdf/wheel.urdf.xacro (robot description, xacro)
@@ -54,5 +54,7 @@
     <transmission name="${fb}_${lr}_wheel_joint_trans">
       <type>transmission_interface/SimpleTransmission</type>
-      <joint name="${fb}_${lr}_wheel_joint" />
+      <joint name="${fb}_${lr}_wheel_joint" type="continuous">
+          <hardwareInterface>EffortJointInterface</hardwareInterface>
+      </joint>
       <actuator name="${fb}_${lr}_wheel_joint_motor">
         <hardwareInterface>EffortJointInterface</hardwareInterface>
