Commit message: Added kinect and joy_teleop

File: labrob_description/urdf/labrob.urdf.xacro (robot description, xacro)
@@ -4,4 +4,5 @@
   <xacro:include filename="$(find labrob_description)/urdf/materials.urdf.xacro" />
   <xacro:include filename="$(find labrob_description)/urdf/wheel.urdf.xacro" />
+  <xacro:include filename="$(find turtlebot_description)/urdf/sensors/kinect.urdf.xacro"/>
   <!-- PROPERTY LIST -->
   <!--All units in m-kg-s-radians unit system -->
@@ -39,5 +40,5 @@
   </gazebo>
   <joint name="base_footprint_joint" type="fixed">
-  <origin xyz="0 0 ${wheel_radius - base_z_origin_to_wheel_origin}" rpy="0 0 0" />
+    <origin xyz="0 0 ${wheel_radius - base_z_origin_to_wheel_origin}" rpy="0 0 0" />
     <parent link="base_footprint"/>
     <child link="base_link" />
@@ -75,4 +76,13 @@
   <wheel fb="back" lr="right" parent="base_link" translateX="-1" translateY="-1" flipY="-1"/>
   <wheel fb="back" lr="left" parent="base_link" translateX="-1" translateY="1" flipY="-1"/>
+  <!-- Kinect -->
+  <link name="kinect_link"/>
+  <joint name="kinect_joint" type="fixed">
+    <origin xyz="0.6 0 -0.1" rpy="0 0 0" />
+    <parent link="base_link"/>
+    <child link="kinect_link" />
+  </joint>
+  <sensor_kinect  parent="kinect_link"/>
+  <!-- Skid steer drive controller -->
   <gazebo>
     <plugin name="skid_steer_drive_controller" filename="libgazebo_ros_skid_steer_drive.so">

File: labrob_description/urdf/materials.urdf.xacro (robot description, xacro)
@@ -1,27 +1,27 @@
 <?xml version="1.0"?>
 <robot>
-	<material name="Black">
-		<color rgba="0.0 0.0 0.0 1.0"/>
-	</material>
-	<material name="Blue">
-		<color rgba="0.0 0.0 0.8 1.0"/>
-	</material>
-	<material name="Green">
-		<color rgba="0.0 0.8 0.0 1.0"/>
-	</material>
-	<material name="Gray">
-		<color rgba="0.7 0.7 0.7 1.0"/>
-	</material>
-	<material name="DarkGray">
-		<color rgba="0.3 0.3 0.3 1.0"/>
-	</material>
-	<material name="Red">
-		<color rgba="0.8 0.0 0.0 1.0"/>
-	</material>
-	<material name="White">
-		<color rgba="1.0 1.0 1.0 1.0"/>
-	</material>
-	<material name="Yellow">
-		<color rgba="0.8 0.8 0.0 1.0"/>
-	</material>
+  <material name="Black">
+    <color rgba="0.0 0.0 0.0 1.0"/>
+  </material>
+  <material name="Blue">
+    <color rgba="0.0 0.0 0.8 1.0"/>
+  </material>
+  <material name="Green">
+    <color rgba="0.0 0.8 0.0 1.0"/>
+  </material>
+  <material name="Gray">
+    <color rgba="0.7 0.7 0.7 1.0"/>
+  </material>
+  <material name="DarkGray">
+    <color rgba="0.3 0.3 0.3 1.0"/>
+  </material>
+  <material name="Red">
+    <color rgba="0.8 0.0 0.0 1.0"/>
+  </material>
+  <material name="White">
+    <color rgba="1.0 1.0 1.0 1.0"/>
+  </material>
+  <material name="Yellow">
+    <color rgba="0.8 0.8 0.0 1.0"/>
+  </material>
 </robot>

Commit message: Added labrob_worlds package

File: labrob_description/urdf/labrob.urdf.xacro (robot description, xacro)
@@ -8,8 +8,11 @@
   <!--All units in m-kg-s-radians unit system -->
   <property name="M_PI" value="3.1415926535897931" />
+  <property name="M_PI_2" value="1.570796327" />
+  <property name="DEG_TO_RAD" value="0.017453293" />
   <!-- Main Body-base -->
   <property name="base_x_size" value="1.0" />
   <property name="base_y_size" value="0.5" />
   <property name="base_z_size" value="0.25" />
+  <property name="hokuyo_size" value="0.05" />
   <property name="base_mass" value="35" /> <!-- in kg-->
   <!--Inertial macros for the box and cylinder. Units are kg*m^2-->
@@ -56,5 +59,5 @@
       <origin xyz="0 0 0" rpy="0 0 0" />
       <geometry>
-        <box size="1 0.5 0.25"/>
+        <box size="${base_x_size} ${base_y_size} ${base_z_size}"/>
       </geometry>
       <material name="Yellow" />
@@ -63,5 +66,5 @@
       <origin xyz="0 0 0" rpy="0 0 0 " />
       <geometry>
-        <box size="1 0.5 0.25"/>
+        <box size="${base_x_size} ${base_y_size} ${base_z_size}"/>
       </geometry>
     </collision>
@@ -76,16 +79,62 @@
   <wheel fb="back" lr="right" parent="base_link" translateX="-1" translateY="-1" flipY="-1"/>
   <wheel fb="back" lr="left" parent="base_link" translateX="-1" translateY="1" flipY="-1"/>
-  <!-- Kinect -->
+  <!-- SENSORS -->
+  <!-- hokuyo -->
+  <link name="hokuyo_link">
+    <visual>
+      <origin xyz="0 0 0" rpy="0 0 0" />
+      <geometry>
+        <box size="${hokuyo_size} ${hokuyo_size} ${hokuyo_size}"/>
+      </geometry>
+      <material name="Blue" />
+    </visual>
+  </link>
+  <joint name="hokuyo_joint" type="fixed">
+    <origin xyz="${base_x_size/2 - hokuyo_size/2} 0 ${base_z_size/2+hokuyo_size/2}" rpy="0 0 0" />
+    <parent link="base_link"/>
+    <child link="hokuyo_link" />
+  </joint>
+  <gazebo reference="hokuyo_link">
+    <material>Gazebo/Blue</material>
+    <turnGravityOff>false</turnGravityOff>
+    <sensor type="ray" name="head_hokuyo_sensor">
+      <pose>${hokuyo_size/2} 0 0 0 0 0</pose>
+      <visualize>false</visualize>
+      <update_rate>40</update_rate>
+      <ray>
+        <scan>
+          <horizontal>
+            <samples>720</samples>
+            <resolution>1</resolution>
+            <min_angle>-1.570796</min_angle>
+            <max_angle>1.570796</max_angle>
+          </horizontal>
+        </scan>
+        <range>
+          <min>0.10</min>
+          <max>10.0</max>
+          <resolution>0.001</resolution>
+        </range>
+      </ray>
+      <plugin name="gazebo_ros_head_hokuyo_controller" filename="libgazebo_ros_laser.so">
+        <topicName>/scan</topicName>
+        <frameName>hokuyo_link</frameName>
+      </plugin>
+    </sensor>
+  </gazebo>
+  <!-- Kinect
   <link name="kinect_link"/>
   <joint name="kinect_joint" type="fixed">
-    <origin xyz="0.6 0 -0.1" rpy="0 0 0" />
+    <origin xyz="0.5 0 -0.1" rpy="0 0 0" />
     <parent link="base_link"/>
     <child link="kinect_link" />
   </joint>
-  <sensor_kinect  parent="kinect_link"/>
+  <sensor_kinect  parent="kinect_link"/> -->
+  <!-- DRIVE CONTROLLERS -->
   <!-- Skid steer drive controller -->
   <gazebo>
+    <plugin name="gazebo_ros_control" filename="libgazebo_ros_control.so" />
     <plugin name="skid_steer_drive_controller" filename="libgazebo_ros_skid_steer_drive.so">
-      <alwaysOn>true</alwaysOn>
+      <alwaysOn>1</alwaysOn>
       <updateRate>100.0</updateRate>
       <leftFrontJoint>front_left_wheel_joint</leftFrontJoint>
@@ -95,5 +144,5 @@
       <wheelSeparation>${base_y_size}</wheelSeparation>
       <wheelDiameter>${2*wheel_radius}</wheelDiameter>
-      <torque>35</torque>
+      <torque>100</torque>
       <broadcastTF>1</broadcastTF>
       <odometryFrame>map</odometryFrame>
@@ -102,5 +151,34 @@
       <robotBaseFrame>base_footprint</robotBaseFrame>
     </plugin>
+  </gazebo>
+  <!-- Differential drive controller
+  <gazebo>
     <plugin name="gazebo_ros_control" filename="libgazebo_ros_control.so" />
-  </gazebo>
+    <plugin name="differential_drive_controller_back" filename="libgazebo_ros_diff_drive.so">
+      <alwaysOn>true</alwaysOn>
+      <updateRate>100.0</updateRate>
+      <leftJoint>back_left_wheel_joint</leftJoint>
+      <rightJoint>back_right_wheel_joint</rightJoint>
+      <wheelSeparation>${base_y_size}</wheelSeparation>
+      <wheelDiameter>${2*wheel_radius}</wheelDiameter>
+      <torque>100</torque>
+      <commandTopic>cmd_vel</commandTopic>
+      <odometryTopic>odom</odometryTopic>
+      <odometryFrame>map</odometryFrame>
+      <robotBaseFrame>base_footprint</robotBaseFrame>
+    </plugin>
+    <plugin name="differential_drive_controller_front" filename="libgazebo_ros_diff_drive.so">
+      <alwaysOn>true</alwaysOn>
+      <updateRate>100.0</updateRate>
+      <leftJoint>front_left_wheel_joint</leftJoint>
+      <rightJoint>front_right_wheel_joint</rightJoint>
+      <wheelSeparation>${base_y_size}</wheelSeparation>
+      <wheelDiameter>${2*wheel_radius}</wheelDiameter>
+      <torque>100</torque>
+      <commandTopic>cmd_vel</commandTopic>
+      <odometryTopic>odom</odometryTopic>
+      <odometryFrame>map</odometryFrame>
+      <robotBaseFrame>base_footprint</robotBaseFrame>
+    </plugin>
+  </gazebo> -->
 </robot>

Commit message: Made it compatible with ROS kinetic

File: labrob_description/urdf/labrob.urdf.xacro (robot description, xacro)
@@ -7,19 +7,19 @@
   <!-- PROPERTY LIST -->
   <!--All units in m-kg-s-radians unit system -->
-  <property name="M_PI" value="3.1415926535897931" />
-  <property name="M_PI_2" value="1.570796327" />
-  <property name="DEG_TO_RAD" value="0.017453293" />
+  <xacro:property name="M_PI" value="3.1415926535897931" />
+  <xacro:property name="M_PI_2" value="1.570796327" />
+  <xacro:property name="DEG_TO_RAD" value="0.017453293" />
   <!-- Main Body-base -->
-  <property name="base_x_size" value="1.0" />
-  <property name="base_y_size" value="0.5" />
-  <property name="base_z_size" value="0.25" />
-  <property name="hokuyo_size" value="0.05" />
-  <property name="base_mass" value="35" /> <!-- in kg-->
+  <xacro:property name="base_x_size" value="1.0" />
+  <xacro:property name="base_y_size" value="0.5" />
+  <xacro:property name="base_z_size" value="0.25" />
+  <xacro:property name="hokuyo_size" value="0.05" />
+  <xacro:property name="base_mass" value="35" /> <!-- in kg-->
   <!--Inertial macros for the box and cylinder. Units are kg*m^2-->
-  <macro name="box_inertia" params="m x y z">
+  <xacro:macro name="box_inertia" params="m x y z">
     <inertia  ixx="${m*(y*y+z*z)/12}" ixy = "0" ixz = "0"
               iyy="${m*(x*x+z*z)/12}" iyz = "0"
               izz="${m*(x*x+z*z)/12}" />
-  </macro>
+  </xacro:macro>
   <!-- BASE-FOOTPRINT -->
   <!-- base_footprint is a fictitious link(frame) that is on the ground right below base_link origin -->
@@ -138,4 +138,5 @@
       <alwaysOn>1</alwaysOn>
       <updateRate>100.0</updateRate>
+      <robotNamespace>/</robotNamespace>
       <leftFrontJoint>front_left_wheel_joint</leftFrontJoint>
       <rightFrontJoint>front_right_wheel_joint</rightFrontJoint>
@@ -150,4 +151,8 @@
       <odometryTopic>odom</odometryTopic>
       <robotBaseFrame>base_footprint</robotBaseFrame>
+      <covariance_x>0.0001</covariance_x>
+      <covariance_y>0.0001</covariance_y>
+      <covariance_z>0.0001</covariance_z>
+      <covariance_yaw>0.0001</covariance_yaw>
     </plugin>
   </gazebo>

File: labrob_description/urdf/wheel.urdf.xacro (robot description, xacro)
@@ -2,15 +2,15 @@
 <robot name="wheel" xmlns:xacro="http://www.ros.org/wiki/xacro">
   <!-- Wheels -->
-  <property name="wheel_radius" value="0.2" />
-  <property name="wheel_height" value="0.1" />
-  <property name="wheel_mass" value="2.5" /> <!-- in kg-->
-  <property name="base_x_origin_to_wheel_origin" value="0.25" />
-  <property name="base_y_origin_to_wheel_origin" value="0.3" />
-  <property name="base_z_origin_to_wheel_origin" value="0.0" />
-  <macro name="cylinder_inertia" params="m r h">
+  <xacro:property name="wheel_radius" value="0.2" />
+  <xacro:property name="wheel_height" value="0.1" />
+  <xacro:property name="wheel_mass" value="2.5" /> <!-- in kg-->
+  <xacro:property name="base_x_origin_to_wheel_origin" value="0.25" />
+  <xacro:property name="base_y_origin_to_wheel_origin" value="0.3" />
+  <xacro:property name="base_z_origin_to_wheel_origin" value="0.0" />
+  <xacro:macro name="cylinder_inertia" params="m r h">
     <inertia  ixx="${m*(3*r*r+h*h)/12}" ixy = "0" ixz = "0"
               iyy="${m*(3*r*r+h*h)/12}" iyz = "0"
               izz="${m*r*r/2}" />
-  </macro>
+  </xacro:macro>
   <xacro:macro name="wheel" params="fb lr parent translateX translateY flipY"> <!--fb : front, back ; lr: left, right -->
     <link name="${fb}_${lr}_wheel">
